File: USB-C_PD_Module/USB-C_PD_Module_Connector_and_Protection.kicad_sch (KiCad schematic)
At the start: 3 parts, among them J1 USB_C_Receptacle_USB2.0_16P, U2 TVS2200DRV, U3 TPD4E02B04DQA

Commit message: Snap to Grid
Parts:
- added U4: TVS2200DRV, Package_SON:WSON-6-1EP_2x2mm_P0.65mm_EP1x1.6mm, symbol Power_Protection:TVS2200DRV
Connections:
- net CC1: now also U3.10 (NC)
- net CC2: now also U3.6 (NC)
- net D+: now also U3.7 (NC)
- net D-: now also U3.9 (NC)
- net GND: now also U4.1 (GND), U4.2 (GND), U4.3 (GND), U4.7 (GND)
- net VBUS: now also U4.4 (IN), U4.5 (IN), U4.6 (IN)
- no-connect marks 7 -> 3

Commit message: Module Basics
Parts:
- J1: footprint Connector_USB:USB_C_Receptacle_GCT_USB4110 -> Connector_USB:USB_C_Receptacle_GCT_USB4105-xx-A_16P_TopMnt_Horizontal
- renumbered U3 to U1, U4 to U3
Changed lines of the file:
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@@
 		(dnp no)
 		(fields_autoplaced yes)
-		(property "Reference" "U3"
+		(property "Reference" "U1"
 			(at 142.24 109.2199 0)
 			(effects
@@
 			(project "USB-C_PD_Module"
 				(path "/e9157937-4343-4473-886a-dab0513dea03/2a8bbf7b-c7ff-4aaf-8d9e-cc20cea6930f"
-					(reference "U3")
+					(reference "U1")
 					(unit 1)
 				)
@@
 		(on_board yes)
 		(dnp no)
-		(property "Reference" "U4"
+		(property "Reference" "U3"
 			(at 209.55 109.2199 0)
 			(effects
@@
 			(project "USB-C_PD_Module"
 				(path "/e9157937-4343-4473-886a-dab0513dea03/2a8bbf7b-c7ff-4aaf-8d9e-cc20cea6930f"
-					(reference "U4")
+					(reference "U3")
 					(unit 1)
 				)
@@
 		(dnp no)
 		(fields_autoplaced yes)
-		(property "Reference" "#PWR026"
+		(property "Reference" "#PWR05"
 			(at 213.36 134.62 0)
 			(effects
@@
 			(project "USB-C_PD_Module"
 				(path "/e9157937-4343-4473-886a-dab0513dea03/2a8bbf7b-c7ff-4aaf-8d9e-cc20cea6930f"
-					(reference "#PWR026")
+					(reference "#PWR05")
 					(unit 1)
 				)
@@
 			)
 		)
-		(property "Footprint" "Connector_USB:USB_C_Receptacle_GCT_USB4110"
+		(property "Footprint" "Connector_USB:USB_C_Receptacle_GCT_USB4105-xx-A_16P_TopMnt_Horizontal"
 			(at 90.17 85.09 0)
 			(effects
