File: USB-C_PD_Module/USB-C_PD_Module_Main_Sheet.kicad_sch (KiCad schematic)
At the start: 20 parts, among them Q1 IRF7328TRPBF, U1 CYPD3177-24LQ

Commit message: Snap to Grid
Parts:
- removed C4, C5: 100n, Capacitor_SMD:C_0805_2012Metric, symbol Device:C
Other:
- moved on the sheet: C8

Commit message: Module Basics
Parts:
- removed R3, R4: 5k1, Resistor_SMD:R_0805_2012Metric, symbol Device:R
- renumbered C6 to C1, C8 to C4, C7 to C5, R2 to R1, R9 to R2, R6 to R3, R5 to R4, R7 to R5, R8 to R6, U1 to U4
Connections:
- net SCL: no longer names the net of U4.13 (HPI_SCL)
- net SDA: no longer names the net of U4.12 (HPI_SDA)
- no-connect marks 3 -> 5
Other:
- moved on the sheet: C5, D1, D2, JP1, Q1A, Q1B, R2, R3, R4, R5, R6
