File: USB-C_PD_Module/USB-C_PD_Module.kicad_pcb (KiCad board)
At the start: 2 copper layers, 25 parts, among them J1 USB_C_Receptacle_USB2.0_16P, J2 Conn_01x10, J3 Conn_01x10, Q1 IRF7328TRPBF, U1 CYPD3177-24LQ, U2 TVS2200DRV, U3 TPD4E02B04DQA

Commit message: Snap to Grid
Parts:
- removed C4, C5: 100n, Capacitor_SMD:C_0805_2012Metric
- added U4: TVS2200DRV, Package_SON:WSON-6-1EP_2x2mm_P0.65mm_EP1x1.6mm, F.Cu at (120.7, 95.2)
- moved J3 131.6 mm to (155.4, 111.4)
- moved J2 129.2 mm to (145.3, 114.0)
- moved R5 122.1 mm to (169.5, 88.3), turned to -90 degrees
- moved R7 120.4 mm to (168.9, 91.4), turned to 180 degrees
- moved U2 118.9 mm to (120.7, 102.2), turned to 90 degrees
- moved R6 118.4 mm to (171.4, 77.5)
- moved Q1 116.3 mm to (177.2, 88.9)
- moved J1 115.6 mm to (114.2, 98.7)
- moved C7 114.3 mm to (170.8, 82.5), turned to 90 degrees
- moved U3 114.1 mm to (120.4, 98.7)
- moved R4 111.3 mm to (152.0, 93.7)
- moved R8 110.7 mm to (161.9, 86.4), turned to 180 degrees
- moved R3 108.9 mm to (146.9, 93.7)
- moved R2 106.8 mm to (141.8, 93.7)
- moved D1 105.0 mm to (172.1, 88.9), turned to -90 degrees
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Connections:
- U3 pad 10: unconnected-(U3-NC-Pad10) -> /USB-C Connector and Protection/CC1
- U3 pad 6: unconnected-(U3-NC-Pad6) -> /USB-C Connector and Protection/CC2
- U3 pad 7: unconnected-(U3-NC-Pad7) -> /USB-C Connector and Protection/D+
- U3 pad 9: unconnected-(U3-NC-Pad9) -> /USB-C Connector and Protection/D-

Commit message: Module Basics
Parts:
- removed the R3 at (146.9, 93.7)
- removed the R4 at (152.0, 93.7)
- J1: footprint Connector_USB:USB_C_Receptacle_GCT_USB4110 -> Connector_USB:USB_C_Receptacle_GCT_USB4105-xx-A_16P_TopMnt_Horizontal
- moved R3 54.3 mm to (124.2, 104.3), turned to 90 degrees
- moved C5 49.6 mm to (126.2, 104.3)
- moved Q1 48.5 mm to (131.1, 104.0), turned to 180 degrees
- moved J3 45.8 mm to (115.6, 88.9), turned to 90 degrees
- moved D1 39.0 mm to (136.1, 104.0), turned to 90 degrees
- moved R4 34.9 mm to (138.7, 104.6), turned to 90 degrees
- moved R2 33.8 mm to (114.7, 91.9)
- moved D2 33.3 mm to (111.4, 91.9)
- moved C1 33.3 mm to (138.0, 97.0), turned to 0 degrees
- moved R5 31.2 mm to (139.3, 101.5), turned to 0 degrees
- moved C3 30.3 mm to (138.0, 94.5), turned to 0 degrees
- moved J2 30.1 mm to (115.6, 109.2), turned to 90 degrees
- moved JP1 29.1 mm to (118.2, 91.9), turned to 0 degrees
- moved R6 28.1 mm to (140.6, 104.6), turned to -90 degrees
- moved C2 27.5 mm to (138.0, 91.9), turned to 0 degrees
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- renumbered C6 to C1, C8 to C4, C7 to C5, R2 to R1, R9 to R2, R6 to R3, R5 to R4, R7 to R5, R8 to R6, U3 to U1, U4 to U3, U1 to U4
Connections:
- J1 pad A6: /USB-C Connector and Protection/D+ -> /D+
- J1 pad A7: /USB-C Connector and Protection/D- -> /D-
- J1 pad B6: /USB-C Connector and Protection/D+ -> /D+
- J1 pad B7: /USB-C Connector and Protection/D- -> /D-
- J3 pad 1: unconnected-(J3-Pin_1-Pad1) -> /Connector/FAULT
- J3 pad 10: unconnected-(J3-Pin_10-Pad10) -> /Connector/VBUS_MIN
- J3 pad 2: unconnected-(J3-Pin_2-Pad2) -> /Connector/FLIP
- J3 pad 3: unconnected-(J3-Pin_3-Pad3) -> /D-
- J3 pad 4: unconnected-(J3-Pin_4-Pad4) -> /D+
- J3 pad 7: unconnected-(J3-Pin_7-Pad7) -> /Connector/ISNK_FINE
- J3 pad 8: unconnected-(J3-Pin_8-Pad8) -> /Connector/ISNK_COARSE
- J3 pad 9: unconnected-(J3-Pin_9-Pad9) -> /Connector/VBUS_MAX
- U1 pad 2: /USB-C Connector and Protection/D- -> /D-
- U1 pad 4: /USB-C Connector and Protection/D+ -> /D+
- U1 pad 7: /USB-C Connector and Protection/D+ -> /D+
- U1 pad 9: /USB-C Connector and Protection/D- -> /D-
- U4 pad 12: /Connector/SDA -> unconnected-(U4-HPI_SDA-Pad12)
- U4 pad 13: /Connector/SCL -> unconnected-(U4-HPI_SCL-Pad13)
Routing:
- net +3V3: track 0.00 -> 33.4 mm, vias 0 -> 2
- net /USB-C Connector and Protection/CC1: track 0.00 -> 25.3 mm, vias 0 -> 2
- net Net-(C5-Pad2): track 0.00 -> 21.4 mm
- net VBUS: track 0.00 -> 21.2 mm
- net /Main Sheet/VBUS_FET_EN: track 0.00 -> 21.0 mm, vias 0 -> 2
- net /Connector/FLIP: track 0.00 -> 19.6 mm
- net /D-: track 0.00 -> 19.1 mm, vias 0 -> 1
- net /Connector/FAULT: track 0.00 -> 18.9 mm, vias 0 -> 2
- net /USB-C Connector and Protection/CC2: track 0.00 -> 18.8 mm, vias 0 -> 2
- net /D+: track 0.00 -> 18.2 mm, vias 0 -> 1
- net GND: track 0.00 -> 12.6 mm, vias 0 -> 12
- net Net-(D1-A): track 0.00 -> 12.3 mm
- net Net-(D1-K): track 0.00 -> 9.03 mm
- net Net-(D2-K): track 0.00 -> 7.87 mm
- net VBUSOUT: track 0.00 -> 7.40 mm, vias 0 -> 18
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- added copper zone on F.Cu, net +3V3
- added copper zone on F.Cu, net Net-(D1-K)
- added copper zone on F.Cu, net VBUS
- added copper zone on F.Cu, net VCCD
Other:
- board outline added: 35.6 x 25.4 mm
- copper layers 2 -> 4

Commit message: Layout Finished
Connections:
- J2 pad 1: unconnected-(J2-Pin_1-Pad1) -> GND
- J2 pad 10: unconnected-(J2-Pin_10-Pad10) -> VBUSOUT
- J2 pad 2: unconnected-(J2-Pin_2-Pad2) -> GND
- J2 pad 3: unconnected-(J2-Pin_3-Pad3) -> GND
- J2 pad 4: unconnected-(J2-Pin_4-Pad4) -> GND
- J2 pad 5: unconnected-(J2-Pin_5-Pad5) -> GND
- J2 pad 6: unconnected-(J2-Pin_6-Pad6) -> VBUSOUT
- J2 pad 7: unconnected-(J2-Pin_7-Pad7) -> VBUSOUT
- J2 pad 8: unconnected-(J2-Pin_8-Pad8) -> VBUSOUT
- J2 pad 9: unconnected-(J2-Pin_9-Pad9) -> VBUSOUT
- J3 pad 5: unconnected-(J3-Pin_5-Pad5) -> GND
- J3 pad 6: unconnected-(J3-Pin_6-Pad6) -> GND
Routing:
- net +3V3: track 33.4 -> 31.7 mm
- net GND: track 12.6 -> 11.5 mm, vias 12 -> 61
- net /USB-C Connector and Protection/CC1: track 25.3 -> 24.6 mm
- net VBUS: track 21.2 -> 21.7 mm
- added copper zone on B.Cu, net GND
- added copper zone on F.Cu, net GND
- added copper zone on In1.Cu, net GND
- added copper zone on In2.Cu, net GND
- added copper zone on B.Cu, net VBUSOUT
- added copper zone on F.Cu, net VBUSOUT
Other:
- board size 35.6 x 25.4 mm -> 35.6 x 20.3 mm
