File: USB-C_PD_Module/USB-C_PD_Module_Connector.kicad_sch (KiCad schematic)
At the start: 2 parts, among them J2 Conn_01x10, J3 Conn_01x10

Commit message: Module Basics
Connections:
- net D+: now also J3.4 (Pin_4)
- net D-: now also J3.3 (Pin_3)
- net FAULT: now also J3.1 (Pin_1)
- net FLIP: now also J3.2 (Pin_2)
- net ISNK_COARSE: now also J3.8 (Pin_8)
- net ISNK_FINE: now also J3.7 (Pin_7)
- net VBUS_MAX: now also J3.9 (Pin_9)
- net VBUS_MIN: now also J3.10 (Pin_10)
Changed lines of the file:
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@@
 		(rev "1.0")
+	)
+	(wire
+		(pts
+			(xy 127 109.22) (xy 132.08 109.22)
+		)
+		(stroke
+			(width 0)
+			(type default)
+		)
+	)
+	(wire
+		(pts
+			(xy 127 93.98) (xy 132.08 93.98)
+		)
+		(stroke
+			(width 0)
+			(type default)
+		)
+	)
+	(wire
+		(pts
+			(xy 127 88.9) (xy 132.08 88.9)
+		)
+		(stroke
+			(width 0)
+			(type default)
+		)
+	)
+	(wire
+		(pts
+			(xy 127 86.36) (xy 132.08 86.36)
+		)
+		(stroke
+			(width 0)
+			(type default)
+		)
+	)
+	(wire
+		(pts
+			(xy 127 106.68) (xy 132.08 106.68)
+		)
+		(stroke
+			(width 0)
+			(type default)
+		)
+	)
+	(wire
+		(pts
+			(xy 127 104.14) (xy 132.08 104.14)
+		)
+		(stroke
+			(width 0)
+			(type default)
+		)
+	)
+	(wire
+		(pts
+			(xy 127 91.44) (xy 132.08 91.44)
+		)
+		(stroke
+			(width 0)
+			(type default)
+		)
+	)
+	(wire
+		(pts
+			(xy 127 101.6) (xy 132.08 101.6)
+		)
+		(stroke
+			(width 0)
+			(type default)
+		)
 	)
 	(hierarchical_label "D-"
 		(shape bidirectional)
-		(at 64.77 125.73 0)
-		(fields_autoplaced yes)
-		(effects
-			(font
-				(size 1.27 1.27)
-			)
-			(justify left)
+		(at 127 91.44 180)
+		(fields_autoplaced yes)
+		(effects
+			(font
+				(size 1.27 1.27)
+			)
+			(justify right)
 		)
 	)
 	(hierarchical_label "VBUS_MAX"
 		(shape output)
-		(at 81.28 119.38 0)
-		(fields_autoplaced yes)
-		(effects
-			(font
-				(size 1.27 1.27)
-			)
-			(justify left)
+		(at 127 106.68 180)
+		(fields_autoplaced yes)
+		(effects
+			(font
+				(size 1.27 1.27)
+			)
+			(justify right)
 		)
 	)
 	(hierarchical_label "FLIP"
 		(shape output)
-		(at 81.28 135.89 0)
-		(fields_autoplaced yes)
-		(effects
-			(font
-				(size 1.27 1.27)
-			)
-			(justify left)
+		(at 127 88.9 180)
+		(fields_autoplaced yes)
+		(effects
+			(font
+				(size 1.27 1.27)
+			)
+			(justify right)
 		)
 	)
 	(hierarchical_label "ISNK_FINE"
 		(shape output)
-		(at 81.28 124.46 0)
-		(fields_autoplaced yes)
-		(effects
-			(font
-				(size 1.27 1.27)
-			)
-			(justify left)
+		(at 127 101.6 180)
+		(fields_autoplaced yes)
+		(effects
+			(font
+				(size 1.27 1.27)
+			)
+			(justify right)
 		)
 	)
 	(hierarchical_label "VBUS_MIN"
 		(shape output)
-		(at 81.28 121.92 0)
-		(fields_autoplaced yes)
-		(effects
-			(font
-				(size 1.27 1.27)
-			)
-			(justify left)
+		(at 127 109.22 180)
+		(fields_autoplaced yes)
+		(effects
+			(font
+				(size 1.27 1.27)
+			)
+			(justify right)
 		)
 	)
 	(hierarchical_label "FAULT"
 		(shape output)
-		(at 81.28 138.43 0)
-		(fields_autoplaced yes)
-		(effects
-			(font
-				(size 1.27 1.27)
-			)
-			(justify left)
-		)
-	)
-	(hierarchical_label "SDA"
-		(shape bidirectional)
-		(at 81.28 133.35 0)
-		(fields_autoplaced yes)
-		(effects
-			(font
-				(size 1.27 1.27)
-			)
-			(justify left)
+		(at 127 86.36 180)
+		(fields_autoplaced yes)
+		(effects
+			(font
+				(size 1.27 1.27)
+			)
+			(justify right)
 		)
 	)
 	(hierarchical_label "ISNK_COARSE"
 		(shape output)
-		(at 81.28 127 0)
-		(fields_autoplaced yes)
-		(effects
-			(font
-				(size 1.27 1.27)
-			)
-			(justify left)
-		)
-	)
-	(hierarchical_label "SCL"
-		(shape input)
-		(at 81.28 130.81 0)
-		(fields_autoplaced yes)
-		(effects
-			(font
-				(size 1.27 1.27)
-			)
-			(justify left)
+		(at 127 104.14 180)
+		(fields_autoplaced yes)
+		(effects
+			(font
+				(size 1.27 1.27)
+			)
+			(justify right)
 		)
 	)
 	(hierarchical_label "D+"
 		(shape bidirectional)
-		(at 64.77 123.19 0)
-		(fields_autoplaced yes)
-		(effects
-			(font
-				(size 1.27 1.27)
-			)
-			(justify left)
+		(at 127 93.98 180)
+		(fields_autoplaced yes)
+		(effects
+			(font
+				(size 1.27 1.27)
+			)
+			(justify right)
 		)
 	)
@@
 	(symbol
 		(lib_id "power:VCCQ")
-		(at 113.03 111.76 0)
+		(at 91.44 120.65 0)
 		(unit 1)
 		(exclude_from_sim no)
@@
 		(dnp no)
 		(fields_autoplaced yes)
-		(property "Reference" "#PWR024"
-			(at 113.03 115.57 0)
+		(property "Reference" "#PWR023"
+			(at 91.44 124.46 0)
 			(effects
 				(font
@@
 		)
 		(property "Value" "VBUSOUT"
-			(at 113.03 106.68 0)
+			(at 91.44 115.57 0)
 			(effects
 				(font
@@
 		)
 		(property "Footprint" ""
-			(at 113.03 111.76 0)
+			(at 91.44 120.65 0)
 			(effects
 				(font
@@
 		)
 		(property "Datasheet" ""
-			(at 113.03 111.76 0)
+			(at 91.44 120.65 0)
 			(effects
 				(font
@@
 		)
 		(property "Description" "Power symbol creates a global label with name \"VCCQ\""
-			(at 113.03 111.76 0)
+			(at 91.44 120.65 0)
 			(effects
 				(font
@@
 			(project "USB-C_PD_Module"
 				(path "/e9157937-4343-4473-886a-dab0513dea03/6cb13895-410c-4d2e-a670-b234d66656a3"
-					(reference "#PWR024")
+					(reference "#PWR023")
 					(unit 1)
 				)
@@
 	(symbol
 		(lib_id "power:GND")
-		(at 113.03 124.46 0)
+		(at 91.44 133.35 0)
 		(unit 1)
 		(exclude_from_sim no)
@@
 		(dnp no)
 		(fields_autoplaced yes)
-		(property "Reference" "#PWR025"
-			(at 113.03 130.81 0)
+		(property "Reference" "#PWR024"
+			(at 91.44 139.7 0)
 			(effects
 				(font
@@
 		)
 		(property "Value" "GND"
-			(at 113.03 129.54 0)
+			(at 91.44 138.43 0)
 			(effects
 				(font
@@
 		)
 		(property "Footprint" ""
-			(at 113.03 124.46 0)
+			(at 91.44 133.35 0)
 			(effects
 				(font
@@
 		)
 		(property "Datasheet" ""
-			(at 113.03 124.46 0)
+			(at 91.44 133.35 0)
 			(effects
 				(font
@@
 		)
 		(property "Description" "Power symbol creates a global label with name \"GND\" , ground"
-			(at 113.03 124.46 0)
+			(at 91.44 133.35 0)
 			(effects
 				(font
@@
 			(project "USB-C_PD_Module"
 				(path "/e9157937-4343-4473-886a-dab0513dea03/6cb13895-410c-4d2e-a670-b234d66656a3"
-					(reference "#PWR025")
+					(reference "#PWR024")
 					(unit 1)
 				)

Commit message: Layout Finished
Connections:
- net GND: now also J2.1 (Pin_1), J2.2 (Pin_2), J2.3 (Pin_3), J2.4 (Pin_4), J2.5 (Pin_5), J3.5 (Pin_5), J3.6 (Pin_6)
- net VBUSOUT: now also J2.10 (Pin_10), J2.6 (Pin_6), J2.7 (Pin_7), J2.8 (Pin_8), J2.9 (Pin_9)
Other:
- moved on the sheet: J2, J3
